Commit message: up to bug1

File: m2wr_description/urdf/m2wr.xacro (robot description, xacro)
@@ -1,9 +1,7 @@
 <?xml version="1.0" ?>
-<robot name="m2wr" xmlns:xacro="https://www.ros.org/wiki/xacro" >
-  <!-- include the xacro files-->
-  <xacro:include filename="$(find m2wr_description)/urdf/material.xacro" />
-  <xacro:include filename="$(find m2wr_description)/urdf/gazebo.xacro" />
-  <xacro:include filename="$(find m2wr_description)/urdf/macro.xacro" />
-<!-- Chassis defined here -->
+<robot name="m2wr" xmlns:xacro="http://www.ros.org/wiki/xacro">
+  <xacro:include filename="$(find m2wr_description)/urdf/materials.xacro" />
+  <xacro:include filename="$(find m2wr_description)/urdf/m2wr.gazebo" />
+  <xacro:include filename="$(find m2wr_description)/urdf/macros.xacro" />
   <link name="link_chassis">
     <!-- pose and inertial -->
@@ -14,4 +12,5 @@
       <inertia ixx="0.0395416666667" ixy="0" ixz="0" iyy="0.106208333333" iyz="0" izz="0.106208333333"/>
     </inertial>
+    <!-- body -->
     <collision name="collision_chassis">
       <geometry>
@@ -49,7 +48,6 @@
       </geometry>
     </visual>
-    </link>
-<!-- Sensor -->
-<link name="sensor_laser">
+  </link>
+  <link name="sensor_laser">
     <inertial>
       <origin xyz="0 0 0" rpy="0 0 0" />
@@ -76,9 +74,7 @@
     <child link="sensor_laser"/>
   </joint>
-  <!-- Left Wheel and right wheel link -->
-   <xacro:link_wheel name="link_right_wheel" />
-   <xacro:link_wheel name="link_left_wheel" />
-  <!--   Joint for left and right wheel  -->
-   <xacro:joint_wheel name="joint_right_wheel"  child="link_right_wheel"  origin_xyz="-0.05 0.15 0"  />
-   <xacro:joint_wheel name="joint_left_wheel"   child="link_left_wheel"   origin_xyz="-0.05 -0.15 0"  />
+  <xacro:link_wheel name="link_right_wheel" />
+  <xacro:joint_wheel name="joint_right_wheel" child="link_right_wheel" origin_xyz="-0.05 0.20 0" />
+  <xacro:link_wheel name="link_left_wheel" />
+  <xacro:joint_wheel name="joint_left_wheel" child="link_left_wheel" origin_xyz="-0.05 -0.20 0" />
 </robot>
